File: AC07_LoRa_Mary/kicad/AC07_LoRa_Mary/AC07_LoRa_Mary.kicad_sch (KiCad schematic)
At the start: 28 parts, among them CN1 Leafony Bus, J1 Conn_Coaxial, U1 CMWX1ZZABZ-091, U2 ATECC608A-MAHDA, U3 TCA9536ADTMR

Commit message: add AC07 layout & sch pdf
Other:
- company: Leafony Systems Ins. -> Leafony Systems Inc.
- title: Leafony LoRa ABZ -> Leafony AC07 LoRa Mary
Changed lines of the file:
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@@
 	(paper "A3")
 	(title_block
-		(title "Leafony LoRa ABZ")
+		(title "Leafony AC07 LoRa Mary")
 		(date "2024-04-24")
-		(rev "v0.2")
-		(company "Leafony Systems Ins.")
+		(rev "v1.2")
+		(company "Leafony Systems Inc.")
 	)
 	(junction
@@
 		)
 		(instances
-			(project "leafony_lora_abz"
+			(project "AC07_LoRa_Mary"
 				(path "/e2743b78-cc59-458c-8fb0-4238f348a49f"
 					(reference "#FLG0102")
@@
 		)
 		(instances
-			(project "leafony_lora_abz"
+			(project "AC07_LoRa_Mary"
 				(path "/e2743b78-cc59-458c-8fb0-4238f348a49f"
 					(reference "#PWR018")
@@
 		)
 		(instances
-			(project "leafony_lora_abz"
+			(project "AC07_LoRa_Mary"
 				(path "/e2743b78-cc59-458c-8fb0-4238f348a49f"
 					(reference "#PWR013")
@@
 		)
 		(instances
-			(project "leafony_lora_abz"
+			(project "AC07_LoRa_Mary"
 				(path "/e2743b78-cc59-458c-8fb0-4238f348a49f"
 					(reference "J1")
@@
 		)
 		(instances
-			(project "leafony_lora_abz"
+			(project "AC07_LoRa_Mary"
 				(path "/e2743b78-cc59-458c-8fb0-4238f348a49f"
 					(reference "C2")
@@
 		)
 		(instances
-			(project "leafony_lora_abz"
+			(project "AC07_LoRa_Mary"
 				(path "/e2743b78-cc59-458c-8fb0-4238f348a49f"
 					(reference "#PWR09")
@@
 		)
 		(instances
-			(project "leafony_lora_abz"
+			(project "AC07_LoRa_Mary"
 				(path "/e2743b78-cc59-458c-8fb0-4238f348a49f"
 					(reference "C5")
@@
 		)
 		(instances
-			(project "leafony_lora_abz"
+			(project "AC07_LoRa_Mary"
 				(path "/e2743b78-cc59-458c-8fb0-4238f348a49f"
 					(reference "#PWR0101")
@@
 		)
 		(instances
-			(project "leafony_lora_abz"
+			(project "AC07_LoRa_Mary"
 				(path "/e2743b78-cc59-458c-8fb0-4238f348a49f"
 					(reference "R3")
@@
 		)
 		(instances
-			(project "leafony_lora_abz"
+			(project "AC07_LoRa_Mary"
 				(path "/e2743b78-cc59-458c-8fb0-4238f348a49f"
 					(reference "#PWR010")
@@
 		)
 		(instances
-			(project "leafony_lora_abz"
+			(project "AC07_LoRa_Mary"
 				(path "/e2743b78-cc59-458c-8fb0-4238f348a49f"
 					(reference "#PWR08")
@@
 		)
 		(instances
-			(project "leafony_lora_abz"
+			(project "AC07_LoRa_Mary"
 				(path "/e2743b78-cc59-458c-8fb0-4238f348a49f"
 					(reference "#PWR06")
@@
 		)
 		(instances
-			(project "leafony_lora_abz"
+			(project "AC07_LoRa_Mary"
 				(path "/e2743b78-cc59-458c-8fb0-4238f348a49f"
 					(reference "#PWR012")
@@
 		)
 		(instances
-			(project "leafony_lora_abz"
+			(project "AC07_LoRa_Mary"
 				(path "/e2743b78-cc59-458c-8fb0-4238f348a49f"
 					(reference "#PWR022")
@@
 		)
 		(instances
-			(project "leafony_lora_abz"
+			(project "AC07_LoRa_Mary"
 				(path "/e2743b78-cc59-458c-8fb0-4238f348a49f"
 					(reference "U1")
@@
 		)
 		(instances
-			(project "leafony_lora_abz"
+			(project "AC07_LoRa_Mary"
 				(path "/e2743b78-cc59-458c-8fb0-4238f348a49f"
 					(reference "C7")
@@
 		)
 		(instances
-			(project "leafony_lora_abz"
+			(project "AC07_LoRa_Mary"
 				(path "/e2743b78-cc59-458c-8fb0-4238f348a49f"
 					(reference "#PWR014")
@@
 		)
 		(instances
-			(project "leafony_lora_abz"
+			(project "AC07_LoRa_Mary"
 				(path "/e2743b78-cc59-458c-8fb0-4238f348a49f"
 					(reference "CN1")
@@
 		)
 		(instances
-			(project "leafony_lora_abz"
+			(project "AC07_LoRa_Mary"
 				(path "/e2743b78-cc59-458c-8fb0-4238f348a49f"
 					(reference "C9")
@@
 		)
 		(instances
-			(project "leafony_lora_abz"
+			(project "AC07_LoRa_Mary"
 				(path "/e2743b78-cc59-458c-8fb0-4238f348a49f"
 					(reference "R8")
@@
 		)
 		(instances
-			(project "leafony_lora_abz"
+			(project "AC07_LoRa_Mary"
 				(path "/e2743b78-cc59-458c-8fb0-4238f348a49f"
 					(reference "#PWR011")
@@
 		)
 		(instances
-			(project "leafony_lora_abz"
+			(project "AC07_LoRa_Mary"
 				(path "/e2743b78-cc59-458c-8fb0-4238f348a49f"
 					(reference "C4")
@@
 		)
 		(instances
-			(project "leafony_lora_abz"
+			(project "AC07_LoRa_Mary"
 				(path "/e2743b78-cc59-458c-8fb0-4238f348a49f"
 					(reference "LOGO1")
@@
 		)
 		(instances
-			(project "leafony_lora_abz"
+			(project "AC07_LoRa_Mary"
 				(path "/e2743b78-cc59-458c-8fb0-4238f348a49f"
 					(reference "#PWR017")
@@
 		)
 		(instances
-			(project "leafony_lora_abz"
+			(project "AC07_LoRa_Mary"
 				(path "/e2743b78-cc59-458c-8fb0-4238f348a49f"
 					(reference "U2")
@@
 		)
 		(instances
-			(project "leafony_lora_abz"
+			(project "AC07_LoRa_Mary"
 				(path "/e2743b78-cc59-458c-8fb0-4238f348a49f"
 					(reference "#PWR019")
@@
 		)
 		(instances
-			(project "leafony_lora_abz"
+			(project "AC07_LoRa_Mary"
 				(path "/e2743b78-cc59-458c-8fb0-4238f348a49f"
 					(reference "#PWR016")
@@
 		)
 		(instances
-			(project "leafony_lora_abz"
+			(project "AC07_LoRa_Mary"
 				(path "/e2743b78-cc59-458c-8fb0-4238f348a49f"
 					(reference "#PWR02")
@@
 		)
 		(instances
-			(project "leafony_lora_abz"
+			(project "AC07_LoRa_Mary"
 				(path "/e2743b78-cc59-458c-8fb0-4238f348a49f"
 					(reference "#PWR015")
@@
 		)
 		(instances
-			(project "leafony_lora_abz"
+			(project "AC07_LoRa_Mary"
 				(path "/e2743b78-cc59-458c-8fb0-4238f348a49f"
 					(reference "C1")
@@
 		)
 		(instances
-			(project "leafony_lora_abz"
+			(project "AC07_LoRa_Mary"
 				(path "/e2743b78-cc59-458c-8fb0-4238f348a49f"
 					(reference "#PWR01")
@@
 		)
 		(instances
-			(project "leafony_lora_abz"
+			(project "AC07_LoRa_Mary"
 				(path "/e2743b78-cc59-458c-8fb0-4238f348a49f"
 					(reference "C10")
@@
 		)
 		(instances
-			(project "leafony_lora_abz"
+			(project "AC07_LoRa_Mary"
 				(path "/e2743b78-cc59-458c-8fb0-4238f348a49f"
 					(reference "#PWR026")
@@
 		)
 		(instances
-			(project "leafony_lora_abz"
+			(project "AC07_LoRa_Mary"
 				(path "/e2743b78-cc59-458c-8fb0-4238f348a49f"
 					(reference "R1")
@@
 		)
 		(instances
-			(project "leafony_lora_abz"
+			(project "AC07_LoRa_Mary"
 				(path "/e2743b78-cc59-458c-8fb0-4238f348a49f"
 					(reference "#PWR024")
@@
 		)
 		(instances
-			(project "leafony_lora_abz"
+			(project "AC07_LoRa_Mary"
 				(path "/e2743b78-cc59-458c-8fb0-4238f348a49f"
 					(reference "R5")
@@
 		)
 		(instances
-			(project "leafony_lora_abz"
+			(project "AC07_LoRa_Mary"
 				(path "/e2743b78-cc59-458c-8fb0-4238f348a49f"
 					(reference "U3")
@@
 		)
 		(instances
-			(project "leafony_lora_abz"
+			(project "AC07_LoRa_Mary"
 				(path "/e2743b78-cc59-458c-8fb0-4238f348a49f"
 					(reference "R4")
@@
 		)
 		(instances
-			(project "leafony_lora_abz"
+			(project "AC07_LoRa_Mary"
 				(path "/e2743b78-cc59-458c-8fb0-4238f348a49f"
 					(reference "C8")
@@
 		)
 		(instances
-			(project "leafony_lora_abz"
+			(project "AC07_LoRa_Mary"
 				(path "/e2743b78-cc59-458c-8fb0-4238f348a49f"
 					(reference "#FLG01")
@@
 		)
 		(instances
-			(project "leafony_lora_abz"
+			(project "AC07_LoRa_Mary"
 				(path "/e2743b78-cc59-458c-8fb0-4238f348a49f"
 					(reference "C12")
@@
 		)
 		(instances
-			(project "leafony_lora_abz"
+			(project "AC07_LoRa_Mary"
 				(path "/e2743b78-cc59-458c-8fb0-4238f348a49f"
 					(reference "#PWR020")
@@
 		)
 		(instances
-			(project "leafony_lora_abz"
+			(project "AC07_LoRa_Mary"
 				(path "/e2743b78-cc59-458c-8fb0-4238f348a49f"
 					(reference "#PWR025")
@@
 		)
 		(instances
-			(project "leafony_lora_abz"
+			(project "AC07_LoRa_Mary"
 				(path "/e2743b78-cc59-458c-8fb0-4238f348a49f"
 					(reference "#PWR05")
@@
 		)
 		(instances
-			(project "leafony_lora_abz"
+			(project "AC07_LoRa_Mary"
 				(path "/e2743b78-cc59-458c-8fb0-4238f348a49f"
 					(reference "TP2")
@@
 		)
 		(instances
-			(project "leafony_lora_abz"
+			(project "AC07_LoRa_Mary"
 				(path "/e2743b78-cc59-458c-8fb0-4238f348a49f"
 					(reference "TP1")
@@
 		)
 		(instances
-			(project "leafony_lora_abz"
+			(project "AC07_LoRa_Mary"
 				(path "/e2743b78-cc59-458c-8fb0-4238f348a49f"
 					(reference "R9")
@@
 		)
 		(instances
-			(project "leafony_lora_abz"
+			(project "AC07_LoRa_Mary"
 				(path "/e2743b78-cc59-458c-8fb0-4238f348a49f"
 					(reference "#PWR07")
@@
 		)
 		(instances
-			(project "leafony_lora_abz"
+			(project "AC07_LoRa_Mary"
 				(path "/e2743b78-cc59-458c-8fb0-4238f348a49f"
 					(reference "C6")
@@
 		)
 		(instances
-			(project "leafony_lora_abz"
+			(project "AC07_LoRa_Mary"
 				(path "/e2743b78-cc59-458c-8fb0-4238f348a49f"
 					(reference "#PWR023")
@@
 		)
 		(instances
-			(project "leafony_lora_abz"
+			(project "AC07_LoRa_Mary"
 				(path "/e2743b78-cc59-458c-8fb0-4238f348a49f"
 					(reference "#PWR021")
@@
 		)
 		(instances
-			(project "leafony_lora_abz"
+			(project "AC07_LoRa_Mary"
 				(path "/e2743b78-cc59-458c-8fb0-4238f348a49f"
 					(reference "#PWR03")
@@
 		)
 		(instances
-			(project "leafony_lora_abz"
+			(project "AC07_LoRa_Mary"
 				(path "/e2743b78-cc59-458c-8fb0-4238f348a49f"
 					(reference "C11")
@@
 		)
 		(instances
-			(project "leafony_lora_abz"
+			(project "AC07_LoRa_Mary"
 				(path "/e2743b78-cc59-458c-8fb0-4238f348a49f"
 					(reference "C3")
@@
 		)
 		(instances
-			(project "leafony_lora_abz"
+			(project "AC07_LoRa_Mary"
 				(path "/e2743b78-cc59-458c-8fb0-4238f348a49f"
 					(reference "R2")
@@
 		)
 		(instances
-			(project "leafony_lora_abz"
+			(project "AC07_LoRa_Mary"
 				(path "/e2743b78-cc59-458c-8fb0-4238f348a49f"
 					(reference "#PWR04")
@@
 		)
 		(instances
-			(project "leafony_lora_abz"
+			(project "AC07_LoRa_Mary"
 				(path "/e2743b78-cc59-458c-8fb0-4238f348a49f"
 					(reference "R6")
